Commit message: try real robot

File: tuto_description/robots/ur_gripper.urdf.xacro (robot description, xacro)
@@ -13,8 +13,8 @@
   <xacro:if value="$(arg ur_enabled)">
     <link name="world" />
-    <joint name="ur_fixed_joint" type="fixed">
+    <joint name="virtual_joint" type="fixed">
       <parent link="world" />
       <child link="base_link" />
-      <origin xyz="0 0.0 0" rpy="0.0 0.0 0.0" />
+      <origin xyz="0 0.0 0.01" rpy="0.0 0.0 0.0" />
     </joint>
     <joint name="ur_real_ee_fixed_joint" type="fixed">

Commit message: marker-update

File: tuto_description/robots/ur_gripper.urdf.xacro (robot description, xacro)
@@ -12,9 +12,15 @@
   <xacro:property name="base_z_size" value="0.55" />
   <xacro:if value="$(arg ur_enabled)">
-    <link name="world" />
-    <joint name="virtual_joint" type="fixed">
+    <link name="real_base_link" />
+    <joint name="real_base_joint" type="fixed">
+      <parent link="real_base_link" />
+      <child link="base_link" />
+      <origin xyz="0 0.0 0.0" rpy="0.0 0.0 ${M_PI}" />
+    </joint>
+    <link name="world"/>
+    <joint name="world_base_joint" type="fixed">
       <parent link="world" />
-      <child link="base_link" />
-      <origin xyz="0 0.0 0.01" rpy="0.0 0.0 0.0" />
+      <child link="real_base_link" />
+      <origin xyz="0 0.0 0.01" rpy="0.0 0.0 0" />
     </joint>
     <joint name="ur_real_ee_fixed_joint" type="fixed">

Commit message: update

File: tuto_description/robots/ur_gripper.urdf.xacro (robot description, xacro)
@@ -6,5 +6,6 @@
   <xacro:property name="M_PI" value="3.14159"/>
   <!--components-->
-  <xacro:include filename="$(find ur_e_description)/urdf/ur5e.urdf.xacro" />
+    <xacro:include filename="$(find ur_e_description)/urdf/ur5e.urdf.xacro" />
+<!--   <xacro:include filename="$(find ur_description)/urdf/ur5.urdf.xacro" /> -->
   <xacro:include filename="$(find robotiq_2f_85_gripper_visualization)/urdf/robotiq_arg2f_85_model_macro.xacro" />
   <xacro:property name="base_x_size" value="0.76" />
@@ -22,5 +23,5 @@
       <parent link="world" />
       <child link="real_base_link" />
-      <origin xyz="0 0.0 0.01" rpy="0.0 0.0 0" />
+      <origin xyz="0 0.0 0.0" rpy="0.0 0.0 0" />
     </joint>
     <joint name="ur_real_ee_fixed_joint" type="fixed">
@@ -31,4 +32,5 @@
     <link name="real_ee_link"/>
     <xacro:ur5e_robot prefix="" joint_limited="false"/>
+    <!-- <xacro:ur5_robot prefix="" joint_limited="false"/> -->
     <!-- gripper -->
     <xacro:if value="$(arg gripper_enabled)">

File: tuto_description/robots/ur_gripper_config.urdf.xacro (robot description, xacro)
@@ -19,5 +19,5 @@
          </geometry>
          <material name="bar1">
-           <color rgba="0 0.5 0 1.0"/>
+           <color rgba="0.192 0.192 0.192 1.0"/>
          </material>
        </visual>
@@ -36,5 +36,5 @@
          </geometry>
          <material name="bar2">
-           <color rgba="0 0.5 0 1.0"/>
+           <color rgba="0.192 0.192 0.192 1.0"/>
          </material>
        </visual>
@@ -53,5 +53,5 @@
          </geometry>
          <material name="bar3">
-           <color rgba="0 0.5 0 1.0"/>
+           <color rgba="0.192 0.192 0.192 1.0"/>
          </material>
        </visual>
@@ -70,5 +70,5 @@
          </geometry>
          <material name="bar4">
-           <color rgba="0 0.5 0 1.0"/>
+           <color rgba="0.192 0.192 0.192 1.0"/>
          </material>
        </visual>
@@ -87,5 +87,5 @@
          </geometry>
          <material name="table">
-           <color rgba="0 0.5 0 1.0"/>
+           <color rgba="0.192 0.192 0.192 1.0"/>
          </material>
        </visual>
